Commit message: New panther_ros simulation software - replacing the description inputs to avoid the sliding effect in the gazebo simulator

File: panther_description/urdf/components/external_antenna.urdf.xacro (robot description, xacro)
@@ -53,23 +53,6 @@
         <sensor name="navsat" type="navsat">
           <plugin filename="ignition-gazebo-navsat-system" name="ignition::gazebo::systems::NavSat" />
-          <ignition_frame_id>gps</ignition_frame_id>
           <always_on>1</always_on>
           <update_rate>5</update_rate>
-          <!-- <gps>
-            <position_sensing>
-              <horizontal>
-                <noise type="gaussian">
-                  <mean>0.0</mean>
-                  <stddev>0.01</stddev>
-                </noise>
-              </horizontal>
-              <vertical>
-                <noise type="gaussian">
-                  <mean>0.0</mean>
-                  <stddev>0.01</stddev>
-                </noise>
-              </vertical>
-            </position_sensing>
-          </gps> -->
         </sensor>
       </gazebo>

File: panther_description/urdf/panther.urdf.xacro (robot description, xacro)
@@ -7,13 +7,13 @@
   <xacro:arg name="imu_pos_y" default="0.025" />
   <xacro:arg name="imu_pos_z" default="0.092" />
-  <xacro:arg name="imu_rot_r" default="3.14" />
-  <xacro:arg name="imu_rot_p" default="-1.57" />
-  <xacro:arg name="imu_rot_y" default="0.0" />
-  <xacro:arg name="use_arm" default="true" />
+  <xacro:arg name="imu_rot_r" default="0.0" />
+  <xacro:arg name="imu_rot_p" default="0.0" />
+  <xacro:arg name="imu_rot_y" default="-1.57" />
+  <xacro:arg name="use_arm" default="false" />
   <xacro:arg name="simulation_engine" default="ignition-gazebo" />
   <xacro:arg name="wheel_config_file"
-    default="$(find panther_description)/config/custom.yaml" />
+    default="$(find panther_description)/config/WH01.yaml" />
   <xacro:arg name="controller_config_file"
-    default="$(find panther_controller)/config/custom_controller.yaml" />
+    default="$(find panther_controller)/config/WH01_controller.yaml" />
   <xacro:arg name="battery_config_file"
     default="$(find panther_description)/config/battery_ign_plugin.yaml" />
@@ -51,18 +51,5 @@
       topic="velodyne_points"
       simulation_engine="$(arg simulation_engine)"  />
-    <!-- Antenna for GPS -->
-  <xacro:include filename="$(find panther_description)/urdf/components/external_antenna.urdf.xacro" ns="antenna" />
-  <xacro:antenna.external_antenna
-    parent_link="base_link"
-    xyz="0.00 0.0 0.640"
-    rpy="0.0 0.0 0.0" />
-  <joint name="base_to_gps_joint" type="fixed">
-      <origin xyz="-0.433 0.0 0.13925"
-        rpy="0.0 0.0 0.0" />
-      <parent link="gps_link" />
-      <child link="base_link" />
-  </joint>
-  <link name="gps_link" />
-    <!-- UR5e arm + Wand Assembly -->
+   <!-- UR5e arm + Wand Assembly -->
     <xacro:property name="use_arm" value="$(arg use_arm)" />
     <xacro:if value="${use_arm}">
@@ -103,4 +90,4 @@
         <origin xyz="0 0 0" rpy="0 0 ${-pi/2}" />
       </xacro:universal_robot.ur_robot>
-    </xacro:if>
+      </xacro:if>
 </robot>
